Commit message: feat: moving robot with teleop

File: ros2_ws/src/galaxea_simulation/urdf/r1_v2_1_0.urdf (robot description, URDF)
Before this commit: robot r1_v2_1_0, 37 links, 36 joints
Joints:
- joint steer_motor_joint1: limit lower=-1.5708 upper=1.5708 effort=44 velocity=3.1416 -> lower=-3.1416 upper=3.1416 effort=44 velocity=3.1416
- joint steer_motor_joint2: limit lower=-1.5708 upper=1.5708 effort=44 velocity=3.1416 -> lower=-3.1416 upper=3.1416 effort=44 velocity=3.1416
- joint steer_motor_joint3: limit lower=-1.5708 upper=1.5708 effort=44 velocity=3.1416 -> lower=-3.1416 upper=3.1416 effort=44 velocity=3.1416
